File: myProject/kicad_pcb.kicad_pcb (KiCad board)
At the start: 2 copper layers, 180 x 180 mm, 145 parts, among them J10 Jack-DC, SW1 SW_DIP_x01, SW10 SW_DIP_x01, SW11 SW_DIP_x01, SW12 SW_DIP_x01, SW13 SW_DIP_x01, SW14 SW_DIP_x01, SW15 SW_DIP_x01, SW16 SW_DIP_x01, SW2 SW_DIP_x01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

Commit message: added gerber and drill files
Parts:
- moved C18 14.2 mm to (68.3, 136.0)
- moved C19 14.2 mm to (87.6, 153.8)
- moved D4 14.2 mm to (92.7, 147.0)
- moved R10 14.2 mm to (74.6, 136.0)
- moved C2 14.2 mm to (111.7, 136.9)
- moved C3 14.2 mm to (111.7, 142.1)
- moved L3 14.2 mm to (81.0, 143.1)
- moved R11 14.2 mm to (74.6, 132.5)
- moved R9 14.2 mm to (75.1, 127.1)
- moved U24 14.2 mm to (102.5, 125.6)
- moved U3 14.2 mm to (104.1, 139.1)
- moved U4 14.2 mm to (86.3, 124.9)
- moved C16 9.62 mm to (90.1, 137.7)
- moved U23 9.12 mm to (162.8, 39.0)
- moved R2 4.93 mm to (102.1, 93.8)
Routing:
- net GND: track 0.00 -> 1329.5 mm, vias 0 -> 22
- net 3V3: track 0.00 -> 1133.2 mm, vias 0 -> 11
- net /Power/VIN_IP: track 0.00 -> 287.7 mm, vias 0 -> 4
- net VDD: track 0.00 -> 209.7 mm, vias 0 -> 3
- net X46: track 0.00 -> 188.5 mm, vias 0 -> 3
- net X44: track 0.00 -> 184.1 mm, vias 0 -> 2
- net X13_BLE_TXD: track 0.00 -> 168.3 mm, vias 0 -> 2
- net X12_BLE_RXD: track 0.00 -> 167.8 mm, vias 0 -> 2
- net X16: track 0.00 -> 146.6 mm
- net X19: track 0.00 -> 143.9 mm
- net X27: track 0.00 -> 143.2 mm
- net X17: track 0.00 -> 142.2 mm, vias 0 -> 2
- net X29: track 0.00 -> 136.4 mm
- net X10: track 0.00 -> 135.6 mm, vias 0 -> 2
- net X9: track 0.00 -> 135.4 mm, vias 0 -> 2
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